Commit message: v2 of robot description (custom sim) now rviz works with meshes

File: team_ws/src/mini_challenge_1/urdf/puzzlebot.xacro (robot description, xacro)
@@ -2,14 +2,11 @@
 <!-- PuzzleBot differential drive -->
 <robot name="puzzlebot" xmlns:xacro="http://www.ros.org/wiki/xacro">
-	<!-- files for gazebo costumization
-	<xacro:include filename="$(find puzzlebot_gazebo)/urdf/materials.xacro" />
-	<xacro:include filename="$(find puzzlebot_gazebo)/urdf/parameters.xacro" />
-	<xacro:include filename="$(find puzzlebot_gazebo)/urdf/puzzlebot.gazebo" />
-	<xacro:include filename="$(find puzzlebot_gazebo)/urdf/macros.xacro" />
-	-->
-	<!-- Dummy link to fiz robot chassis -->
+	<!-- ================ URDF VARIABLES ================ -->
+	<xacro:property name="PI" value="3.1415926535897931"/>
+	<!-- ================ DUMMY LINK TO FIX CHASIS ================ -->
   	<link name="puzzlebot_frame">
 		<pose>0 0 0 0 0 0</pose>
 	</link>
+	<!-- ================ CHASIS ================ -->
 	<joint name="base_link_to_chassis" type="fixed">
 		<parent link="puzzlebot_frame"/>
@@ -19,40 +16,39 @@
 		<pose>0 0 0 0 0 0</pose>
 		<visual>
-			<!-- box only -->
-			<origin xyz="0 0 0" rpy="0 0 0"/>
-			<geometry>
-				<box size="0.3 0.2 0.15"/>
-			</geometry>
-			<!-- with mesh  -->
-			<!--
 			<origin xyz="0 0 0" rpy="${PI/2} 0 ${PI/2}"/>
 			<geometry>
-				<mesh filename="file://${mesh_chassis}"/>
+				<mesh filename="file://$(find mini_challenge_1)/meshes/MCR2_1000_13_Chassis.stl"/>
 			</geometry>
-			-->
 		</visual>
-		<!--
-		<collision name="collision_chassis">
-			<origin rpy="0 0 0" xyz="0 0 0"/>
+	</link>
+	<!-- ================ RIGHT WHEEL ================ -->
+	<joint name="base_to_right_w" type="continuous">
+		<parent link="chassis" />
+		<child link="right_wheel" />
+		<origin xyz="0.05 -0.09 0.0" />
+		<axis xyz="0 1 0" rpy="0 0 0" />
+	</joint>
+	<link name="right_wheel">
+		<pose>0 0 0 0 0 0</pose>
+		<visual>
+			<origin xyz="0 0 0" rpy="-${PI/2} 0 0" />
 			<geometry>
-					<box size="${chassisX} ${chassisY} ${chassisZ}"/>
+				<mesh filename="file://$(find mini_challenge_1)/meshes/MCR2_1000_1_1_Wheel_Coupler_2.stl"/>
 			</geometry>
-		</collision>
-		<inertial>
-		<mass value="${chassisMass}"/>
-		<xacro:box_inertia m="${chassisMass}" x="${chassisX}" y="${chassisY}" z="${chassisZ}" />
-		</inertial>
-		-->
-	<!-- agregar caster wheel en frame -->
-		<collision>
-			<origin xyz="-0.095 0 -0.0425" rpy="0 0 0"/>
+		</visual>
+	</link>
+	<!-- ================ RIGHT WHEEL ================ -->
+	<joint name="base_to_left_w" type="continuous">
+		<parent link="chassis" />
+		<child link="left_wheel" />
+		<origin xyz="0.05 0.09 0.0" />
+		<axis xyz="0 1 0" rpy="0 0 0" />
+	</joint>
+	<link name="left_wheel">
+		<pose>0 0 0 0 0 0</pose>
+		<visual>
+			<origin xyz="0 0 0" rpy="${PI/2} 0 0" />
 			<geometry>
-				<sphere radius="0.1"/>
-			</geometry>
-		</collision>
-		<visual>
-			<origin xyz="-0.095 0 -0.0425" rpy="0 0 0"/>
-			<geometry>
-				<sphere radius="0.1"/>
+				<mesh filename="file://$(find mini_challenge_1)/meshes/MCR2_1000_1_1_Wheel_Coupler_2.stl"/>
 			</geometry>
 		</visual>

Commit message: cambio de frames en el urdf a map -> baselink -> left_wheel/right_wheel, con movimiento en las ruedas

File: team_ws/src/mini_challenge_1/urdf/puzzlebot.xacro (robot description, xacro)
@@ -4,14 +4,13 @@
 	<!-- ================ URDF VARIABLES ================ -->
 	<xacro:property name="PI" value="3.1415926535897931"/>
-	<!-- ================ DUMMY LINK TO FIX CHASIS ================ -->
-  	<link name="puzzlebot_frame">
-		<pose>0 0 0 0 0 0</pose>
+	<!-- ******   Base-Link   ****** -->
+	<link name="map">
 	</link>
 	<!-- ================ CHASIS ================ -->
 	<joint name="base_link_to_chassis" type="fixed">
-		<parent link="puzzlebot_frame"/>
-		<child link="chassis"/>
+		<parent link="map"/>
+		<child link="base_link"/>
 	</joint>
-	<link name="chassis">
+	<link name="base_link">
 		<pose>0 0 0 0 0 0</pose>
 		<visual>
@@ -24,5 +23,5 @@
 	<!-- ================ RIGHT WHEEL ================ -->
 	<joint name="base_to_right_w" type="continuous">
-		<parent link="chassis" />
+		<parent link="base_link" />
 		<child link="right_wheel" />
 		<origin xyz="0.05 -0.09 0.0" />
@@ -40,5 +39,5 @@
 	<!-- ================ RIGHT WHEEL ================ -->
 	<joint name="base_to_left_w" type="continuous">
-		<parent link="chassis" />
+		<parent link="base_link" />
 		<child link="left_wheel" />
 		<origin xyz="0.05 0.09 0.0" />
